File: DCBLmotor_Driver_Unite/Daughter_Board.brd (EAGLE design)
At the start: 53.5 x 50.6 mm, 40 parts, among them CN1 FX23L-20P-0.5SV12, CN2 DF63-2P-3.96DSA, CN4 DF63-3P-3.96DSA, IC1 ACS780KLRTR-150B-T, IC4 DRV8320SRTVT, IC6 LTM8050IY#PBF-ND

Commit message: Temp Commit
Parts:
- added DC1: YFF15PC1C104MT000N, TDK:YFF15PC
Connections:
- new net N$9: DC1.P$1, IC1.P$1
- net +5V: now also DC1.P$2
- net GND: now also DC1.P$3, DC1.P$4, IC1.P$2
Routing:
- net +5V: track 10.8 -> 28.7 mm, vias 0 -> 1
- net GND: track 43.0 -> 52.3 mm, vias 13 -> 14
- net N$9: track 0.00 -> 1.48 mm
- net CU1: track 17.5 -> 16.4 mm
Other:
- board text added: "Caution This board has jeopardy of critical error"
- board text removed: "It's First version functionally test board Have a possibility of a undiscovered fatal malfunction"
Changed lines of the file:
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@@
 <setting verticaltext="up"/>
 </settings>
-<grid distance="2" unitdist="mil" unit="mil" style="lines" multiple="1" display="no" altdistance="5" altunitdist="mil" altunit="mm"/>
+<grid distance="1" unitdist="mil" unit="mil" style="lines" multiple="1" display="no" altdistance="5" altunitdist="mil" altunit="mm"/>
 <layers>
 <layer number="1" name="Top" color="4" fill="1" visible="yes" active="yes"/>
-<layer number="2" name="Route2" color="1" fill="3" visible="yes" active="yes"/>
-<layer number="3" name="Route3" color="4" fill="3" visible="yes" active="yes"/>
+<layer number="2" name="Route2" color="1" fill="3" visible="no" active="yes"/>
+<layer number="3" name="Route3" color="4" fill="3" visible="no" active="yes"/>
 <layer number="4" name="Route4" color="1" fill="4" visible="no" active="no"/>
 <layer number="5" name="Route5" color="4" fill="4" visible="no" active="no"/>
@@
 <layer number="14" name="Route14" color="1" fill="6" visible="no" active="no"/>
 <layer number="15" name="Route15" color="4" fill="6" visible="no" active="no"/>
-<layer number="16" name="Bottom" color="1" fill="1" visible="yes" active="yes"/>
+<layer number="16" name="Bottom" color="1" fill="1" visible="no" active="yes"/>
 <layer number="17" name="Pads" color="2" fill="1" visible="yes" active="yes"/>
 <layer number="18" name="Vias" color="2" fill="1" visible="yes" active="yes"/>
@@
 <layer number="20" name="Dimension" color="24" fill="1" visible="yes" active="yes"/>
 <layer number="21" name="tPlace" color="7" fill="1" visible="yes" active="yes"/>
-<layer number="22" name="bPlace" color="7" fill="1" visible="yes" active="yes"/>
+<layer number="22" name="bPlace" color="7" fill="1" visible="no" active="yes"/>
 <layer number="23" name="tOrigins" color="15" fill="1" visible="yes" active="yes"/>
-<layer number="24" name="bOrigins" color="15" fill="1" visible="yes" active="yes"/>
+<layer number="24" name="bOrigins" color="15" fill="1" visible="no" active="yes"/>
 <layer number="25" name="tNames" color="7" fill="1" visible="yes" active="yes"/>
-<layer number="26" name="bNames" color="7" fill="1" visible="yes" active="yes"/>
-<layer number="27" name="tValues" color="7" fill="1" visible="yes" active="yes"/>
-<layer number="28" name="bValues" color="7" fill="1" visible="yes" active="yes"/>
+<layer number="26" name="bNames" color="7" fill="1" visible="no" active="yes"/>
+<layer number="27" name="tValues" color="7" fill="1" visible="no" active="yes"/>
+<layer number="28" name="bValues" color="7" fill="1" visible="no" active="yes"/>
 <layer number="29" name="tStop" color="7" fill="3" visible="no" active="yes"/>
 <layer number="30" name="bStop" color="7" fill="6" visible="no" active="yes"/>
@@
 <layer number="38" name="bTest" color="7" fill="1" visible="no" active="yes"/>
 <layer number="39" name="tKeepout" color="4" fill="11" visible="yes" active="yes"/>
-<layer number="40" name="bKeepout" color="1" fill="11" visible="yes" active="yes"/>
+<layer number="40" name="bKeepout" color="1" fill="11" visible="no" active="yes"/>
 <layer number="41" name="tRestrict" color="4" fill="10" visible="yes" active="yes"/>
-<layer number="42" name="bRestrict" color="1" fill="10" visible="yes" active="yes"/>
+<layer number="42" name="bRestrict" color="1" fill="10" visible="no" active="yes"/>
 <layer number="43" name="vRestrict" color="2" fill="10" visible="no" active="yes"/>
-<layer number="44" name="Drills" color="7" fill="1" visible="yes" active="yes"/>
+<layer number="44" name="Drills" color="7" fill="1" visible="no" active="yes"/>
 <layer number="45" name="Holes" color="7" fill="1" visible="yes" active="yes"/>
 <layer number="46" name="Milling" color="3" fill="1" visible="no" active="yes"/>
@@
 <layer number="49" name="Reference" color="7" fill="1" visible="no" active="yes"/>
 <layer number="51" name="tDocu" color="7" fill="1" visible="yes" active="yes"/>
-<layer number="52" name="bDocu" color="7" fill="1" visible="yes" active="yes"/>
+<layer number="52" name="bDocu" color="7" fill="1" visible="no" active="yes"/>
 <layer number="88" name="SimResults" color="9" fill="1" visible="no" active="no"/>
 <layer number="89" name="SimProbes" color="9" fill="1" visible="no" active="no"/>
@@
 <wire x1="24.693" y1="67.619" x2="24.693" y2="22.619" width="2.54" layer="21"/>
 <hole x="27.813" y="64.643" drill="2"/>
-<text x="64.15473125" y="49.826834375" size="1.016" layer="21" rot="R210">It's First version functionally test board
-Have a possibility of a undiscovered
-fatal malfunction</text>
 <text x="55.805946875" y="52.57386875" size="1.4224" layer="22" rot="MR30">CAUTION</text>
 <dimension x1="68" y1="22" x2="68" y2="68" x3="82" y3="45" textsize="1.778" layer="1"/>
@@
 <dimension x1="48" y1="24" x2="48" y2="35" x3="17" y3="29.5" textsize="1.778" layer="1"/>
 <text x="66.9544" y="64.5668" size="0.4064" layer="21" rot="R90">+3.3V</text>
+<text x="41.529" y="32.5374" size="1.778" layer="21" rot="R90">Caution
+This board has jeopardy
+of critical error</text>
 </plain>
 <attributes>
@@
 <element name="R8" library="Panasonic" package="R0805" value="ERA-6AEB5762V" x="67.056" y="40.259" rot="MR270"/>
 <element name="IC1" library="ACS780" package="7-PIN_PSOP" value="ACS780KLRTR-150B-T" x="45.1096" y="35.6508" rot="R90"/>
+<element name="DC1" library="TDK" package="YFF15PC" value="YFF15PC1C104MT000N" x="49.5808" y="34.0614"/>
 </elements>
 <signals>
@@
 <wire x1="57.2008" y1="63.891521875" x2="57.2008" y2="63.4492" width="0.1524" layer="1"/>
 <via x="57.2008" y="63.4492" extent="1-16" drill="0.25"/>
+<contactref element="IC1" pad="P$2"/>
+<contactref element="DC1" pad="P$4"/>
+<contactref element="DC1" pad="P$3"/>
+<wire x1="47.6096" y1="35.6508" x2="49.9364" y2="35.6508" width="0.1524" layer="1"/>
+<wire x1="49.9364" y1="35.6508" x2="50.506" y2="35.6508" width="0.1524" layer="1"/>
+<wire x1="50.506" y1="35.6508" x2="53.6956" y2="32.4612" width="0.1524" layer="1"/>
+<via x="53.6956" y="32.4612" extent="1-16" drill="0.35"/>
+<wire x1="49.5808" y1="34.3114" x2="49.5808" y2="33.8114" width="0.1524" layer="1"/>
+<wire x1="49.5808" y1="34.3114" x2="49.5808" y2="35.2952" width="0.1524" layer="1"/>
+<wire x1="49.5808" y1="35.2952" x2="49.9364" y2="35.6508" width="0.1524" layer="1"/>
 <wire x1="58.95159375" y1="65.642315625" x2="58.985709375" y2="65.6082" width="0" layer="19" extent="1-1"/>
 </signal>
@@
 <wire x1="47.6096" y1="37.2508" x2="49.668" y2="37.2508" width="0.1524" layer="1"/>
 <wire x1="49.668" y1="37.2508" x2="50.6476" y2="36.2712" width="0.1524" layer="1"/>
-<wire x1="50.6476" y1="36.2712" x2="50.6476" y2="29.4132" width="0.1524" layer="1"/>
-<wire x1="50.6476" y1="29.4132" x2="51.816" y2="28.2448" width="0.1524" layer="1"/>
-<wire x1="51.816" y1="28.2448" x2="54.0512" y2="28.2448" width="0.1524" layer="1"/>
-<wire x1="54.0512" y1="28.2448" x2="54.9656" y2="27.3304" width="0.1524" layer="1"/>
-<wire x1="54.9656" y1="27.3304" x2="54.9254" y2="27.2902" width="0.1524" layer="1"/>
-<wire x1="54.9254" y1="27.2902" x2="54.9254" y2="25.3488" width="0.1524" layer="1"/>
+<wire x1="50.6476" y1="36.2712" x2="52.6288" y2="34.29" width="0.1524" layer="1"/>
+<wire x1="52.6288" y1="34.29" x2="53.086" y2="34.29" width="0.1524" layer="1"/>
+<wire x1="53.086" y1="34.29" x2="54.3052" y2="33.0708" width="0.1524" layer="1"/>
+<wire x1="54.3052" y1="25.969" x2="54.9254" y2="25.3488" width="0.1524" layer="1"/>
+<wire x1="54.3052" y1="33.0708" x2="54.3052" y2="25.969" width="0.1524" layer="1"/>
 </signal>
 <signal name="VCC">
@@
 <wire x1="58.4962" y1="35.9156" x2="58.813" y2="35.9156" width="1.016" layer="16"/>
 <wire x1="58.813" y1="35.9156" x2="61.0228" y2="33.7058" width="1.016" layer="16"/>
+<contactref element="DC1" pad="P$2"/>
+<wire x1="50.0808" y1="34.0614" x2="50.9778" y2="33.1644" width="0.1524" layer="1"/>
+<wire x1="50.9778" y1="33.1644" x2="50.9778" y2="28.8036" width="0.1524" layer="1"/>
+<via x="50.9778" y="28.8036" extent="1-16" drill="0.35"/>
+<wire x1="50.9778" y1="28.8036" x2="51.562" y2="28.2194" width="0.1524" layer="16"/>
+<wire x1="59.271" y1="28.2194" x2="61.9254" y2="30.8738" width="0.1524" layer="16"/>
+<wire x1="51.562" y1="28.2194" x2="59.271" y2="28.2194" width="0.1524" layer="16"/>
 </signal>
 <signal name="N$1">
@@
 <wire x1="41.87" y1="48.6" x2="41.1332" y2="49.7332" width="0" layer="19" extent="1-1"/>
 </signal>
+<signal name="N$9">
+<contactref element="DC1" pad="P$1"/>
+<contactref element="IC1" pad="P$1"/>
+<wire x1="47.6096" y1="34.0508" x2="49.0702" y2="34.0508" width="0.1524" layer="1"/>
+<wire x1="49.0702" y1="34.0508" x2="49.0808" y2="34.0614" width="0.1524" layer="1"/>
+</signal>
 </signals>
