File: DCBLmotor_Driver_Unite/Daughter_Board.sch (EAGLE design)
At the start: 40 parts, among them CN1 FX23L-20P-0.5SV12, CN2 DF63-2P-3.96DSA, CN4 DF63-3P-3.96DSA, IC1 ACS780KLRTR-150B-T, IC4 DRV8320SRTVT, IC6 LTM8050IY#PBF-ND

Commit message: Temp Commit
Parts:
- added DC1: YFF15PC1C104MT000N, TDK:YFF15PC1C104MT000N
Connections:
- new net N$9: DC1.P$1, IC1.VCC
- net +5V: now also DC1.P$2
- net GND: now also DC1.GND, IC1.GND
Other:
- moved on the sheet: C6, PMC3
Changed lines of the file:
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@@
 <part name="R8" library="Panasonic" deviceset="ERA-6AEB5762V" device=""/>
 <part name="IC1" library="ACS780" deviceset="ACS780KLRTR-150B-T" device=""/>
+<part name="DC1" library="TDK" deviceset="YFF15PC1C104MT000N" device=""/>
 </parts>
 <sheets>
@@
 <instance part="C4" gate="G$1" x="104.14" y="99.06"/>
 <instance part="C5" gate="G$1" x="144.78" y="53.34"/>
-<instance part="C6" gate="G$1" x="254" y="7.62"/>
+<instance part="C6" gate="G$1" x="190.5" y="7.62"/>
 <instance part="SUPPLY7" gate="GND" x="132.08" y="-220.98"/>
 <instance part="PMC1" gate="G$1" x="109.22" y="88.9"/>
 <instance part="PMC2" gate="G$1" x="149.86" y="43.18"/>
-<instance part="PMC3" gate="G$1" x="259.08" y="-2.54"/>
+<instance part="PMC3" gate="G$1" x="195.58" y="-2.54"/>
 <instance part="R1" gate="G$1" x="30.48" y="104.14"/>
 <instance part="R2" gate="G$1" x="25.4" y="58.42"/>
@@
 <instance part="R7" gate="G$1" x="-170.18" y="-20.32" rot="R90"/>
 <instance part="R8" gate="G$1" x="-165.1" y="12.7" rot="R90"/>
-<instance part="IC1" gate="G$1" x="299.72" y="-182.88"/>
+<instance part="IC1" gate="G$1" x="233.68" y="-182.88"/>
+<instance part="DC1" gate="G$1" x="254" y="-187.96"/>
 </instances>
 <busses>
@@
 <pinref part="SUPPLY7" gate="GND" pin="GND"/>
 <wire x1="132.08" y1="-218.44" x2="132.08" y2="-215.9" width="0.1524" layer="91"/>
-<wire x1="132.08" y1="-215.9" x2="287.02" y2="-215.9" width="0.1524" layer="91"/>
-<wire x1="287.02" y1="-215.9" x2="287.02" y2="-185.42" width="0.1524" layer="91"/>
+<wire x1="132.08" y1="-215.9" x2="220.98" y2="-215.9" width="0.1524" layer="91"/>
+<wire x1="220.98" y1="-215.9" x2="220.98" y2="-185.42" width="0.1524" layer="91"/>
 </segment>
 <segment>
@@
 <wire x1="-124.46" y1="-147.32" x2="-142.24" y2="-147.32" width="0.1524" layer="91"/>
 <junction x="-142.24" y="-147.32"/>
-<wire x1="-147.32" y1="-139.7" x2="-147.32" y2="-142.24" width="0.1524" layer="91"/>
-<junction x="-147.32" y="-142.24"/>
 <pinref part="CN2" gate="G$1" pin="1"/>
 </segment>
@@
 <label x="-53.34" y="-43.18" size="1.778" layer="95" rot="R90"/>
 </segment>
+<segment>
+<pinref part="IC1" gate="G$1" pin="GND"/>
+<wire x1="246.38" y1="-182.88" x2="259.08" y2="-182.88" width="0.1524" layer="91"/>
+<label x="256.54" y="-182.88" size="1.778" layer="95"/>
+</segment>
+<segment>
+<pinref part="DC1" gate="G$1" pin="GND"/>
+<wire x1="254" y1="-191.08" x2="254" y2="-198.12" width="0.1524" layer="91"/>
+<label x="254" y="-198.12" size="1.778" layer="95"/>
+</segment>
 </net>
 <net name="+3.3V" class="0">
@@
 <pinref part="R2" gate="G$1" pin="2"/>
 <wire x1="20.32" y1="58.42" x2="10.16" y2="58.42" width="0.1524" layer="91"/>
+<label x="10.16" y="58.42" size="1.778" layer="95"/>
 </segment>
 <segment>
@@
 <segment>
 <pinref part="IC1" gate="G$1" pin="VOUT"/>
-<wire x1="312.42" y1="-177.8" x2="325.12" y2="-177.8" width="0.1524" layer="91"/>
+<wire x1="246.38" y1="-177.8" x2="259.08" y2="-177.8" width="0.1524" layer="91"/>
+<label x="256.54" y="-177.8" size="1.778" layer="95"/>
 </segment>
 </net>
@@
 <pinref part="C5" gate="G$1" pin="1"/>
 <pinref part="C6" gate="G$1" pin="1"/>
-<wire x1="254" y1="10.16" x2="254" y2="48.26" width="0.1524" layer="91"/>
-<wire x1="254" y1="48.26" x2="177.8" y2="48.26" width="0.1524" layer="91"/>
+<wire x1="190.5" y1="10.16" x2="190.5" y2="48.26" width="0.1524" layer="91"/>
+<wire x1="190.5" y1="48.26" x2="177.8" y2="48.26" width="0.1524" layer="91"/>
 <junction x="177.8" y="48.26"/>
 <pinref part="PMC2" gate="G$1" pin="1"/>
 <wire x1="149.86" y1="45.72" x2="149.86" y2="154.94" width="0.1524" layer="91"/>
 <pinref part="PMC3" gate="G$1" pin="1"/>
-<wire x1="259.08" y1="0" x2="259.08" y2="53.34" width="0.1524" layer="91"/>
-<wire x1="259.08" y1="53.34" x2="177.8" y2="53.34" width="0.1524" layer="91"/>
+<wire x1="195.58" y1="0" x2="195.58" y2="53.34" width="0.1524" layer="91"/>
+<wire x1="195.58" y1="53.34" x2="177.8" y2="53.34" width="0.1524" layer="91"/>
 <junction x="177.8" y="53.34"/>
 <pinref part="PMC1" gate="G$1" pin="1"/>
@@
 <wire x1="-144.78" y1="30.48" x2="-137.16" y2="30.48" width="0.1524" layer="91"/>
 <wire x1="-137.16" y1="30.48" x2="-137.16" y2="38.1" width="0.1524" layer="91"/>
+<label x="-137.16" y="35.56" size="1.778" layer="95"/>
 </segment>
 </net>
@@
 <wire x1="-48.26" y1="60.96" x2="-40.64" y2="60.96" width="0.1524" layer="91"/>
 </segment>
+<segment>
+<pinref part="DC1" gate="G$1" pin="P$2"/>
+<wire x1="259.08" y1="-187.96" x2="264.16" y2="-187.96" width="0.1524" layer="91"/>
+<label x="264.16" y="-187.96" size="1.778" layer="95"/>
+</segment>
 </net>
 <net name="N$1" class="0">
@@
 <net name="LOSIDE" class="0">
 <segment>
-<wire x1="177.8" y1="-200.66" x2="236.22" y2="-205.74" width="0.1524" layer="91"/>
-<wire x1="236.22" y1="-205.74" x2="236.22" y2="-208.28" width="0.1524" layer="91"/>
+<wire x1="177.8" y1="-200.66" x2="177.8" y2="-208.28" width="0.1524" layer="91"/>
 <wire x1="91.44" y1="-208.28" x2="104.14" y2="-208.28" width="0.1524" layer="91"/>
 <wire x1="104.14" y1="-208.28" x2="109.22" y2="-208.28" width="0.1524" layer="91"/>
@@
 <pinref part="C4" gate="G$1" pin="2"/>
 <wire x1="144.78" y1="-208.28" x2="149.86" y2="-208.28" width="0.1524" layer="91"/>
-<wire x1="149.86" y1="-208.28" x2="236.22" y2="-208.28" width="0.1524" layer="91"/>
+<wire x1="149.86" y1="-208.28" x2="177.8" y2="-208.28" width="0.1524" layer="91"/>
 <wire x1="104.14" y1="93.98" x2="104.14" y2="-208.28" width="0.1524" layer="91"/>
 <pinref part="C6" gate="G$1" pin="2"/>
-<wire x1="177.8" y1="-200.66" x2="254" y2="-203.2" width="0.1524" layer="91"/>
-<wire x1="254" y1="-203.2" x2="254" y2="2.54" width="0.1524" layer="91"/>
+<wire x1="177.8" y1="-200.66" x2="190.5" y2="-200.66" width="0.1524" layer="91"/>
+<wire x1="190.5" y1="-200.66" x2="190.5" y2="2.54" width="0.1524" layer="91"/>
 <junction x="177.8" y="-200.66"/>
 <pinref part="C5" gate="G$1" pin="2"/>
@@
 <wire x1="149.86" y1="-208.28" x2="149.86" y2="38.1" width="0.1524" layer="91"/>
 <pinref part="PMC3" gate="G$1" pin="2"/>
-<wire x1="236.22" y1="-205.74" x2="259.08" y2="-205.74" width="0.1524" layer="91"/>
-<wire x1="259.08" y1="-205.74" x2="259.08" y2="-7.62" width="0.1524" layer="91"/>
-<junction x="236.22" y="-205.74"/>
+<wire x1="177.8" y1="-208.28" x2="195.58" y2="-208.28" width="0.1524" layer="91"/>
+<wire x1="195.58" y1="-208.28" x2="195.58" y2="-7.62" width="0.1524" layer="91"/>
+<junction x="177.8" y="-208.28"/>
 <pinref part="FD2" gate="G$1" pin="A"/>
 <wire x1="91.44" y1="-208.28" x2="91.44" y2="-160.02" width="0.1524" layer="91"/>
@@
 <junction x="144.78" y="-208.28"/>
 <pinref part="IC1" gate="G$1" pin="IP+"/>
-<wire x1="287.02" y1="-180.34" x2="281.94" y2="-180.34" width="0.1524" layer="91"/>
-<wire x1="281.94" y1="-180.34" x2="281.94" y2="-210.82" width="0.1524" layer="91"/>
-<wire x1="281.94" y1="-210.82" x2="132.08" y2="-210.82" width="0.1524" layer="91"/>
+<wire x1="220.98" y1="-180.34" x2="215.9" y2="-180.34" width="0.1524" layer="91"/>
+<wire x1="215.9" y1="-180.34" x2="215.9" y2="-210.82" width="0.1524" layer="91"/>
+<wire x1="215.9" y1="-210.82" x2="132.08" y2="-210.82" width="0.1524" layer="91"/>
 <wire x1="132.08" y1="-109.22" x2="121.92" y2="-109.22" width="0.1524" layer="91"/>
 <wire x1="177.8" y1="-60.96" x2="165.1" y2="-60.96" width="0.1524" layer="91"/>
@@
 </segment>
 </net>
+<net name="N$9" class="0">
+<segment>
+<pinref part="DC1" gate="G$1" pin="P$1"/>
+<pinref part="IC1" gate="G$1" pin="VCC"/>
+<wire x1="248.92" y1="-187.96" x2="246.38" y2="-187.96" width="0.1524" layer="91"/>
+</segment>
+</net>
