File: DCBLmotor_Driver_Unite/Main_bord.brd (EAGLE design)
At the start: 33 x 46 mm, 46 parts, among them CN1 FX23L-20S-0.5SV, CN8 BM11B-SRSS-TB, IC1 TMPM370FYFG, IC2 TMPM373FWDUG, IC5 LTC2862A, SW1 CVS-02TB, SW2 EVQ-PE104K

Commit message: Main_borad is Almost_finshed
Parts:
- removed 0R1, 0R2: 5106, Keystone:5106JUMP_0805
- removed C1, C2: C2012X7R1A475M125AC, TDK:C2012
- removed CN8: BM11B-SRSS-TB, JST:BM11B-SRSS-TB
- removed CR1, CR2, CR3, CR4, CR9: C0816X7R1, TDK:C0816
- removed CR12, CR6, CR7: NSI50010YT1G, ON Semiconductor:SOD-123
- removed DC3, DC4, DC5: YFF21PC1E104MT000N, TDK:YFF21PC
- removed DC6, DC7: YFF15PC1C104MT000N, TDK:YFF15PC
- removed R6, R7: CRCW06031K00JNEAC, VISHAY:0603
- removed RA1: EXB-38V103JV, Pana_Chip_RA:EXB-38V,28V
- removed S2: 220AMA16R, 220AMA16R:220AMA16R
- removed VR2: 3314J-1-104E, Bourns:3314J-1
- added CN2: FTSH-105-01-F-DV-K, FTSH-105-01-F-DV-K:SAMTEC_FTSH-105-01-L-DV
- added R1, R3, R4: MCR006, ROHM:MCR006
- added R5: CRCW06031K00JNEAC, VISHAY:0603
- CN9: value (none) -> DF11-4DP-2DSR; device jst-xh:B4B-XH-A -> Hirose:DF11_4DP-2D
- DC1, DC2: value YFF21PC1E104MT000N -> YFF15PC1C104MT000N; device TDK:YFF21PC -> TDK:YFF15PC
- IC1: value TMPM370FYFG -> ADP3338AKCZ-3.3RL7; device TOSHIBA:LQFP100-P-1414-0.50H -> ADP3338AKCZ-3.3RL7:SOT230P700X180-4N
- SW1: value CVS-02TB -> CVS-01TB; device Nidec:CVS-02B -> Nidec:CVS-01B
- moved LED1 74.6 mm to (3.88, 25.6), turned to 90 degrees
- moved SW1 66.7 mm to (29.2, 26.7), turned to 180 degrees
- moved R2 55.9 mm to (15.0, 17.1)
- moved SW2 53.4 mm to (9.69, 16.7)
- moved DC1 46.5 mm to (23.4, 18.7), turned to 0 degrees
- moved DC2 43.8 mm to (16.2, 19.2), flipped to the top, turned to 180 degrees
- moved L1 42.4 mm to (16.8, 15.1), turned to 0 degrees
- moved IC5 42.4 mm to (2.80, 37.1)
- moved R8 42.4 mm to (3.08, 34.4)
- moved DC15 42.4 mm to (5.28, 37.1)
- moved CN9 39.5 mm to (5.23, 30.6), turned to 270 degrees
- moved IC1 29.0 mm to (14.4, 42.0), turned to 0 degrees
- moved LED3 27.1 mm to (10.7, 24.1), turned to 0 degrees
- moved CR5 24.2 mm to (13.5, 24.1), turned to 90 degrees
- moved XTAL1 4.70 mm to (4.09, 19.5)
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Connections:
- removed net 1U_H: IC1.P$22
- removed net 1U_L: IC1.P$23
- removed net 1V_H: IC1.P$24
- removed net 1V_L: IC1.P$25
- removed net 1W_H: IC1.P$26
- removed net 1W_L: IC1.P$27
- removed net 2U_H: IC1.P$37
- removed net 2U_L: IC1.P$38
- removed net 2V_H: IC1.P$39
- removed net 2V_L: IC1.P$42
- removed net 2W_H: IC1.P$43
- removed net 2W_L: IC1.P$44
- removed net AGND: CR9.P$2, DC2.GND1, DC2.GND2, IC1.P$97
- removed net CU1_1: IC1.P$96
- removed net CU1_2: IC1.P$95
- removed net CU1_3: IC1.P$94
- removed net CU2_1: IC1.P$85
- removed net CU2_2: IC1.P$84
- removed net CU2_3: IC1.P$83
- removed net CVR1: IC1.P$100, VR2.P$2
- removed net CVR2: IC1.P$99
- removed net DIP1: IC1.P$80, RA1.P$5, S2.1
- removed net DIP2: IC1.P$79, RA1.P$8, S2.4
- removed net DIP4: IC1.P$78, RA1.P$6, S2.3
- removed net DIP8: IC1.P$77, RA1.P$7, S2.6
- removed net DVSS(1): IC2.10
- removed net DVSS(2): IC2.28
- removed net EMG1: IC1.P$28
- removed net EMG2: IC1.P$45
- removed net ENC_A-1: IC1.P$30
- removed net ENC_A-2: IC1.P$52
- removed net ENC_B-1: IC1.P$31
- removed net ENC_B-2: IC1.P$53
- removed net ENC_Z-1: IC1.P$32
- removed net ENC_Z-2: IC1.P$54
- removed net LED1_1: CR6.P$C, IC1.P$12
- removed net LED1_2: CR12.P$C, IC1.P$13
- removed net LED1_3: CR7.P$C, IC1.P$15
- removed net LED2_1: IC1.P$16
- removed net LED2_2: IC1.P$17
- removed net LED2_3: IC1.P$18
- removed net N$13: IC1.P$36
- removed net N$14: DC6.P$1, IC1.P$87
- removed net N$15: DC7.P$1, IC1.P$82
- removed net N$16: IC1.P$1
- removed net N$17: IC1.P$35
- removed net N$18: CN8.P$5, IC1.P$67
- removed net N$19: CN8.P$6, IC1.P$66
- removed net N$20: CN8.P$9, IC1.P$63
- removed net N$21: CN8.P$7, IC1.P$65
- removed net N$22: CN8.P$8, IC1.P$64
- removed net N$23: CN8.P$4, IC1.P$68
- removed net N$24: CN8.P$3, IC1.P$69
- removed net N$25: CN8.P$2, IC1.P$70
- removed net N$26: IC1.P$34
- removed net N$27: IC1.P$33
- removed net N$37: CR7.P$A, LED1.P$4
- removed net N$38: CR12.P$A, LED1.P$5
- removed net N$39: CR6.P$A, LED1.P$6
- removed net N$44: 0R2.P$1, CN9.2
- removed net N$46: 0R1.P$1, CN9.1
- removed net N$8: C1.P$1, IC1.P$55
- removed net N$9: C2.P$1, IC1.P$60
- removed net RVDD5: IC2.32
- removed net RX0: IC1.P$11, IC5.P$4
- removed net STBY: IC1.P$9
- removed net SW1: IC1.P$76, R6.P$2, SW1.P$1-1
- removed net SW2: IC1.P$75, R7.P$2, SW1.P$2-1
- removed net TX0: IC1.P$10, IC5.P$1
- new net +3.3V: IC1.2, IC1.4
- new net BOOT: IC2.12, R5.P$2, SW1.P$2-2
- new net CU1: CN1.1, IC2.37
- new net HIN1: CN1.19, IC2.2
- new net HIN2: CN1.16, IC2.4
- new net HIN3: CN1.18, IC2.6
- new net LED_1: IC2.17, R4.P$2
- new net LED_2: IC2.18, R3.P$2
- new net LED_3: IC2.19, R1.P$2
- new net LIN1: CN1.15, IC2.3
- new net LIN2: CN1.20, IC2.5
- new net LIN3: CN1.17, IC2.7
- new net N$31: CN2.7
- new net N$32: CN2.9
- new net RXD1: IC2.46, IC5.P$4
- new net TCK: CN2.4, IC2.15
- new net TDI: CN2.8, IC2.13
- new net TDO: CN2.6, IC2.14
- new net TMS: CN2.2, IC2.16
- new net TXD1: IC2.47, IC5.P$1
- net +5V: now also CN1.25, CN2.1, CN9.P$2, DC8.P$2, DC9.P$1, IC1.1, R2.P$1, R5.P$1; no longer 0R2.P$2, CN8.P$1, CR1.P$1, CR2.P$1, CR3.P$1, CR4.P$1, CR9.P$1, DC1.P$1, DC3.P$2, DC4.P$2, DC5.P$1, R6.P$1, R7.P$1, RA1.P$1, RA1.P$2, RA1.P$3, RA1.P$4
- net A*: now also CN9.P$3; no longer CN9.3
- net AVDD: now also DC1.P$2; no longer DC6.P$2, DC7.P$2, VR2.P$1
- net B*: now also CN9.P$4; no longer CN9.4
- net GND: now also C5.P$2, C6.P$2, CN1.24, CN2.3, CN2.5, CN9.P$1, DC1.P$3, DC1.P$4, DC2.P$3, DC2.P$4, DC8.P$3, DC8.P$4, DC9.P$3, DC9.P$4, IC1.3, IC2.10, IC2.28, IC2.31, IC2.42, SW1.P$2-1; no longer 0R1.P$2, C1.P$2, C2.P$2, CR1.P$2, CR2.P$2, CR3.P$2, CR4.P$2, DC1.GND1, DC1.GND2, DC3.GND1, DC3.GND2, DC4.GND1, DC4.GND2, DC5.GND1, DC5.GND2, DC6.P$3, DC6.P$4, DC7.P$3, DC7.P$4, IC1.P$19, IC1.P$41, IC1.P$48, IC1.P$56, IC1.P$57, IC1.P$62, IC1.P$81, IC1.P$86, S2.2, S2.5, SW1.P$1-2, SW1.P$2-2, VR2.P$3
- net N$1: now also DC2.P$1, IC2.32; no longer DC5.P$2, IC1.P$40
- net N$2: now also DC1.P$1, IC2.43; no longer DC4.P$1, IC1.P$58
- net N$3: now also LED1.P$5, R3.P$1; no longer DC3.P$1, IC1.P$61
- net N$4: now also LED1.P$4, R1.P$1; no longer DC2.P$1, IC1.P$98
- net N$5: now also LED1.P$6, R4.P$1; no longer DC1.P$2, IC1.P$14
- net RESET: now also CN2.10, IC2.34; no longer CN8.P$10, IC1.P$59
- net RS_DIR: now also IC2.48; no longer IC1.P$8
- net VCC: now also CN1.23; no longer R2.P$1
- net X1: no longer IC1.P$47
- net X2: no longer IC1.P$49
Routing:
- net ENC_Z-2: track 113.2 -> 0.00 mm, vias 1 -> 0
- net 2V_H: track 51.9 -> 0.00 mm, vias 1 -> 0
- net ENC_Z-1: track 51.6 -> 0.00 mm, vias 1 -> 0
- net RXD1: track 0.00 -> 51.4 mm, vias 0 -> 2
- net ENC_A-2: track 51.3 -> 0.00 mm
- net 2V_L: track 51.0 -> 0.00 mm, vias 1 -> 0
- net ENC_B-2: track 50.1 -> 0.00 mm
- net 2W_H: track 49.8 -> 0.00 mm, vias 1 -> 0
- net ENC_B-1: track 49.0 -> 0.00 mm, vias 1 -> 0
- net TXD1: track 0.00 -> 48.6 mm, vias 0 -> 2
- net TX0: track 48.5 -> 0.00 mm, vias 4 -> 0
- net RX0: track 46.0 -> 0.00 mm, vias 2 -> 0
- net ENC_A-1: track 45.1 -> 0.00 mm, vias 1 -> 0
- net LED2_1: track 43.6 -> 0.00 mm, vias 2 -> 0
- net 2U_H: track 42.8 -> 0.00 mm, vias 1 -> 0
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- added copper zone on layer 1, net +3.3V
- removed copper zone on layer 1, net GND
- removed copper zone on layer 16, net GND
Other:
- outline, holes or cut-outs redrawn
- board text added: "Boot mode"
- board text removed: "+"
- board text removed: "Adjust of emergency threshold"
- board text removed: "All Transfer port is not isolated"
- board text removed: "CAN FD"
- board text removed: "CAUTION"
- board text removed: "Designed by Ozawa"
- board text removed: "ENC 1"
- board text removed: "ENC 2"
- board text removed: "Hall 1"
- board text removed: "Hall 2"
- board text removed: "It's First version functionally of test board Have a possibility of a undiscovered fatal malfunction"
- board text removed: "It's First version of functionally test board Have a possibility of a undiscovered fatal malfunction"
- board text removed: "MAX +20V"
- board text removed: "Motor 1"
- board text removed: "Motor 2"
- board text removed: "Pilot LED"
- board text removed: "Prototype Ver.1"
- board text removed: "RS485"
- board text removed: "RS485 Power jumper"
- board text removed: "UESR LED"

Commit message: Temp Commit
Parts:
- added CN3: DF11-16DP-2DSA, Hirose:DF11-16DP-2D
- moved C3 35.0 mm to (4.59, 51.8)
- moved C4 35.0 mm to (3.59, 57.3)
- moved C5 35.0 mm to (20.8, 55.2)
- moved C6 35.0 mm to (20.8, 53.7)
- moved CN1 35.0 mm to (20.7, 42.9)
- moved CN2 35.0 mm to (20.7, 42.9)
- moved CN9 35.0 mm to (5.23, 65.6)
- moved CR5 35.0 mm to (13.5, 59.1)
- moved DC1 35.0 mm to (23.4, 53.7)
- moved DC15 35.0 mm to (5.28, 72.1)
- moved DC2 35.0 mm to (16.2, 54.2)
- moved DC8 35.0 mm to (20.4, 57.2)
- moved DC9 35.0 mm to (24.1, 57.2)
- moved IC1 35.0 mm to (14.4, 77.0)
- moved IC2 35.0 mm to (22.3, 55.0)
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